Commit message: add a smile for big wheels!

File: urdf/car.urdf (robot description, URDF)
Before this commit: robot car_robot, 10 links, 9 joints
Links:
- added link eyebrow-left-link; visual box size=0.003 0.018 0.003
- added link eyebrow-right-link; visual box size=0.003 0.018 0.003
- added link smile-link; visual mesh filename=package://car_robot/meshes/smile.stl scale=1 1 1
- link eye-left-link: geometry visual sphere radius=0.009
- link eye-right-link: geometry visual sphere radius=0.009
- link pupil-left-link: geometry visual sphere radius=0.005
- link pupil-right-link: geometry visual sphere radius=0.005
Joints:
- added joint joint-eyebrow-left: type fixed, parent chassis-link, child eyebrow-left-link, origin xyz=0.102 0.028 0.022 rpy=0 0 0
- added joint joint-eyebrow-right: type fixed, parent chassis-link, child eyebrow-right-link, origin xyz=0.102 -0.028 0.022 rpy=0 0 0
- added joint joint-smile: type fixed, parent chassis-link, child smile-link, origin xyz=0.101 0.0 0.0 rpy=0 0 0
- joint joint-eye-left: origin xyz=0.102 0.03 0.01 rpy=0 0 0 -> xyz=0.102 0.028 0.005 rpy=0 0 0
- joint joint-eye-right: origin xyz=0.102 -0.03 0.01 rpy=0 0 0 -> xyz=0.102 -0.028 0.005 rpy=0 0 0
- joint joint-pupil-left: origin xyz=0.005 0 0 rpy=0 0 0 -> xyz=0.006 -0.003 0.004 rpy=0 0 0
- joint joint-pupil-right: origin xyz=0.005 0 0 rpy=0 0 0 -> xyz=0.006 0.003 0.004 rpy=0 0 0
